File: hardware/TheHardGuys_WristWatch/TheHardGuys_WristWatch.kicad_sch (KiCad schematic)
At the start: 0 parts

Commit message: Added ESP32 symbol and footprints
Parts:
- added U1: ~, ESP32_30pin, symbol esp32_30pin_revised:ESP32_30Pin
Changed lines of the file:
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@@
 	(generator_version "9.0")
 	(paper "A4")
+	(symbol
+		(lib_id "esp32_30pin_revised:ESP32_30Pin")
+		(at 146.05 97.79 270)
+		(unit 1)
+		(exclude_from_sim no)
+		(in_bom yes)
+		(on_board yes)
+		(dnp no)
+		(fields_autoplaced yes)
+		(property "Reference" "U1"
+			(at 146.05 66.04 90)
+			(effects
+				(font
+					(size 1.27 1.27)
+				)
+			)
+		)
+		(property "Value" "~"
+			(at 146.05 68.58 90)
+			(effects
+				(font
+					(size 1.27 1.27)
+				)
+			)
+		)
+		(property "Footprint" "ESP32_30pin"
+			(at 146.05 71.12 90)
+			(effects
+				(font
+					(size 1.27 1.27)
+					(color 194 194 0 1)
+				)
+			)
+		)
+		(property "Datasheet" ""
+			(at 146.05 97.79 0)
+			(effects
+				(font
+					(size 1.27 1.27)
+				)
+				(hide yes)
+			)
+		)
+		(property "Description" ""
+			(at 146.05 97.79 0)
+			(effects
+				(font
+					(size 1.27 1.27)
+				)
+				(hide yes)
+			)
+		)
+		(pin "25"
+		)
+		(pin "30"
+		)
+		(pin "15"
+		)
+		(pin "28"
+		)
+		(pin "27"
+		)
+		(pin "12"
+		)
+		(pin "14"
+		)
+		(pin "13"
+		)
+		(pin "29"
+		)
+		(pin "26"
+		)
+		(pin "11"
+		)
+		(pin "22"
+		)
+		(pin "18"
+		)
+		(pin "4"
+		)
+		(pin "2"
+		)
+		(pin "1"
+		)
+		(pin "19"
+		)
+		(pin "21"
+		)
+		(pin "8"
+		)
+		(pin "7"
+		)
+		(pin "20"
+		)
+		(pin "24"
+		)
+		(pin "23"
+		)
+		(pin "5"
+		)
+		(pin "6"
+		)
+		(pin "16"
+		)
+		(pin "10"
+		)
+		(pin "3"
+		)
+		(pin "17"
+		)
+		(pin "9"
+		)
+		(instances
+			(project ""
+				(path "/2f8b587e-5655-46c3-a754-1864bf3bb2c9"
+					(reference "U1")
+					(unit 1)
+				)
+			)
+		)
+	)
 	(sheet_instances
 		(path "/"
